File: Hardware/Boje.sch (EAGLE design)
At the start: 10 parts, among them IC1 TINY13V-10PU, J1 332-02, J2 332-02

Commit message: Board Update
Parts:
- added J3: SWITCH, con-garry:332-02
- J1: value 332-02 -> POWER
- J2: value 332-02 -> Free
Connections:
- new net N$1: J1-1.S, J3-1.S
- net VCC-5V: now also J3-2.S; no longer J1-1.S
Other:
- moved on the sheet: J1-1, J2-2
Changed lines of the file:
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@@
 <part name="R1" library="resistor" deviceset="R-EU_" device="M2012" value="68"/>
 <part name="LDR1" library="rcl" deviceset="R-EU_" device="V526-0" value="LDR"/>
-<part name="J1" library="con-garry" deviceset="332-02" device=""/>
-<part name="J2" library="con-garry" deviceset="332-02" device=""/>
+<part name="J1" library="con-garry" deviceset="332-02" device="" value="POWER"/>
+<part name="J2" library="con-garry" deviceset="332-02" device="" value="Free"/>
+<part name="J3" library="con-garry" deviceset="332-02" device="" value="SWITCH"/>
 </parts>
 <sheets>
@@
 <instances>
 <instance part="IC1" gate="G$1" x="45.72" y="38.1"/>
-<instance part="P+2" gate="VCC" x="22.86" y="55.88"/>
+<instance part="P+2" gate="VCC" x="22.86" y="63.5"/>
 <instance part="GND8" gate="1" x="22.86" y="0"/>
 <instance part="D3" gate="G$1" x="17.78" y="15.24"/>
@@
 <instance part="R1" gate="G$1" x="7.62" y="25.4" rot="R90"/>
 <instance part="LDR1" gate="G$1" x="2.54" y="25.4" rot="R90"/>
-<instance part="J1" gate="-1" x="17.78" y="50.8" rot="R180"/>
+<instance part="J1" gate="-1" x="10.16" y="50.8" rot="R180"/>
 <instance part="J1" gate="-2" x="27.94" y="5.08"/>
 <instance part="J2" gate="-1" x="27.94" y="7.62"/>
-<instance part="J2" gate="-2" x="17.78" y="45.72" rot="R180"/>
+<instance part="J2" gate="-2" x="10.16" y="45.72" rot="R180"/>
+<instance part="J3" gate="-1" x="15.24" y="55.88" rot="R90"/>
+<instance part="J3" gate="-2" x="17.78" y="55.88" rot="R90"/>
 </instances>
 <busses>
@@
 <pinref part="P+2" gate="VCC" pin="VCC"/>
 <wire x1="25.4" y1="50.8" x2="22.86" y2="50.8" width="0.1524" layer="91"/>
-<wire x1="22.86" y1="50.8" x2="22.86" y2="53.34" width="0.1524" layer="91"/>
-<pinref part="J1" gate="-1" pin="S"/>
-<wire x1="22.86" y1="50.8" x2="20.32" y2="50.8" width="0.1524" layer="91"/>
+<wire x1="22.86" y1="50.8" x2="22.86" y2="60.96" width="0.1524" layer="91"/>
+<wire x1="22.86" y1="50.8" x2="17.78" y2="50.8" width="0.1524" layer="91"/>
 <junction x="22.86" y="50.8"/>
+<wire x1="17.78" y1="53.34" x2="17.78" y2="50.8" width="0.1524" layer="91"/>
+<pinref part="J3" gate="-2" pin="S"/>
 </segment>
 </net>
@@
 <pinref part="IC1" gate="G$1" pin="PB1/PCINT1/AIN1/OC0B/INT0/MISO"/>
 <pinref part="J2" gate="-2" pin="S"/>
-<wire x1="25.4" y1="45.72" x2="20.32" y2="45.72" width="0.1524" layer="91"/>
+<wire x1="25.4" y1="45.72" x2="12.7" y2="45.72" width="0.1524" layer="91"/>
 </segment>
 </net>
+<net name="N$1" class="0">
+<segment>
+<pinref part="J1" gate="-1" pin="S"/>
+<pinref part="J3" gate="-1" pin="S"/>
+<wire x1="15.24" y1="50.8" x2="15.24" y2="53.34" width="0.1524" layer="91"/>
+<wire x1="15.24" y1="50.8" x2="12.7" y2="50.8" width="0.1524" layer="91"/>
+</segment>
+</net>

Commit message: Part Change
Parts:
- IC1: value TINY13V-10PU -> AT-TINY85V
Changed lines of the file:
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@@
 </classes>
 <parts>
-<part name="IC1" library="atmel" deviceset="TINY13" device="PU" technology="V-10"/>
+<part name="IC1" library="atmel" deviceset="TINY13" device="PU" technology="V-10" value="AT-TINY85V"/>
 <part name="P+2" library="supply1" deviceset="VCC" device=""/>
 <part name="GND8" library="supply1" deviceset="GND" device=""/>

Commit message: New Layout
Parts:
- removed J3: SWITCH, con-garry:332-02
- added SW1: SWS001, smd-special:SWS001
- D1: value (none) -> LED0
- D2: value (none) -> LED1
- D3: value (none) -> LED2
Connections:
- removed net VCC-5V: IC1.VCC, J3-2.S
- new net VCC: IC1.VCC, SW1.1
- net N$1: now also SW1.2; no longer J3-1.S
Other:
- moved on the sheet: J1-1
Changed lines of the file:
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@@
 <classes>
 <class number="0" name="default" width="0" drill="0">
+<clearance class="0" value="0.205"/>
 </class>
 </classes>
@@
 <part name="P+2" library="supply1" deviceset="VCC" device=""/>
 <part name="GND8" library="supply1" deviceset="GND" device=""/>
-<part name="D3" library="SparkFun-LED" deviceset="LED" device="5MM"/>
-<part name="D2" library="SparkFun-LED" deviceset="LED" device="5MM"/>
-<part name="D1" library="SparkFun-LED" deviceset="LED" device="5MM"/>
+<part name="D3" library="SparkFun-LED" deviceset="LED" device="5MM" value="LED2"/>
+<part name="D2" library="SparkFun-LED" deviceset="LED" device="5MM" value="LED1"/>
+<part name="D1" library="SparkFun-LED" deviceset="LED" device="5MM" value="LED0"/>
 <part name="R3" library="resistor" deviceset="R-EU_" device="M2012" value="68"/>
 <part name="R2" library="resistor" deviceset="R-EU_" device="M2012" value="68"/>
@@
 <part name="J1" library="con-garry" deviceset="332-02" device="" value="POWER"/>
 <part name="J2" library="con-garry" deviceset="332-02" device="" value="Free"/>
-<part name="J3" library="con-garry" deviceset="332-02" device="" value="SWITCH"/>
+<part name="SW1" library="smd-special" deviceset="SWS001" device=""/>
 </parts>
 <sheets>
@@
 <instance part="R1" gate="G$1" x="7.62" y="25.4" rot="R90"/>
 <instance part="LDR1" gate="G$1" x="2.54" y="25.4" rot="R90"/>
-<instance part="J1" gate="-1" x="10.16" y="50.8" rot="R180"/>
+<instance part="J1" gate="-1" x="2.54" y="50.8" rot="R180"/>
 <instance part="J1" gate="-2" x="27.94" y="5.08"/>
 <instance part="J2" gate="-1" x="27.94" y="7.62"/>
 <instance part="J2" gate="-2" x="10.16" y="45.72" rot="R180"/>
-<instance part="J3" gate="-1" x="15.24" y="55.88" rot="R90"/>
-<instance part="J3" gate="-2" x="17.78" y="55.88" rot="R90"/>
+<instance part="SW1" gate="G$1" x="15.24" y="50.8" rot="R90"/>
 </instances>
 <busses>
@@
 </segment>
 </net>
-<net name="VCC-5V" class="0">
+<net name="VCC" class="0">
 <segment>
 <pinref part="IC1" gate="G$1" pin="VCC"/>
@@
 <wire x1="25.4" y1="50.8" x2="22.86" y2="50.8" width="0.1524" layer="91"/>
 <wire x1="22.86" y1="50.8" x2="22.86" y2="60.96" width="0.1524" layer="91"/>
-<wire x1="22.86" y1="50.8" x2="17.78" y2="50.8" width="0.1524" layer="91"/>
+<wire x1="22.86" y1="50.8" x2="20.32" y2="50.8" width="0.1524" layer="91"/>
 <junction x="22.86" y="50.8"/>
-<wire x1="17.78" y1="53.34" x2="17.78" y2="50.8" width="0.1524" layer="91"/>
-<pinref part="J3" gate="-2" pin="S"/>
+<pinref part="SW1" gate="G$1" pin="1"/>
 </segment>
 </net>
@@
 <segment>
 <pinref part="J1" gate="-1" pin="S"/>
-<pinref part="J3" gate="-1" pin="S"/>
-<wire x1="15.24" y1="50.8" x2="15.24" y2="53.34" width="0.1524" layer="91"/>
-<wire x1="15.24" y1="50.8" x2="12.7" y2="50.8" width="0.1524" layer="91"/>
+<wire x1="7.62" y1="50.8" x2="5.08" y2="50.8" width="0.1524" layer="91"/>
+<pinref part="SW1" gate="G$1" pin="2"/>
 </segment>
 </net>
@@
 </sheet>
 </sheets>
-<errors>
-</errors>
 </schematic>
 </drawing>

Commit message: Gerber
Parts:
- removed SW1: SWS001, smd-special:SWS001
- added J3: SWITCH, con-garry:332-02
Connections:
- net N$1: now also J3-1.S; no longer SW1.2
- net VCC: now also J3-2.S; no longer SW1.1
Other:
- moved on the sheet: J1-1
Changed lines of the file:
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@@
 <part name="J1" library="con-garry" deviceset="332-02" device="" value="POWER"/>
 <part name="J2" library="con-garry" deviceset="332-02" device="" value="Free"/>
-<part name="SW1" library="smd-special" deviceset="SWS001" device=""/>
+<part name="J3" library="con-garry" deviceset="332-02" device="" value="SWITCH"/>
 </parts>
 <sheets>
@@
 <instance part="R1" gate="G$1" x="7.62" y="25.4" rot="R90"/>
 <instance part="LDR1" gate="G$1" x="2.54" y="25.4" rot="R90"/>
-<instance part="J1" gate="-1" x="2.54" y="50.8" rot="R180"/>
+<instance part="J1" gate="-1" x="7.62" y="53.34" rot="R180"/>
 <instance part="J1" gate="-2" x="27.94" y="5.08"/>
 <instance part="J2" gate="-1" x="27.94" y="7.62"/>
 <instance part="J2" gate="-2" x="10.16" y="45.72" rot="R180"/>
-<instance part="SW1" gate="G$1" x="15.24" y="50.8" rot="R90"/>
+<instance part="J3" gate="-1" x="12.7" y="58.42" rot="R90"/>
+<instance part="J3" gate="-2" x="17.78" y="58.42" rot="R90"/>
 </instances>
 <busses>
@@
 <pinref part="P+2" gate="VCC" pin="VCC"/>
 <wire x1="25.4" y1="50.8" x2="22.86" y2="50.8" width="0.1524" layer="91"/>
-<wire x1="22.86" y1="50.8" x2="22.86" y2="60.96" width="0.1524" layer="91"/>
-<wire x1="22.86" y1="50.8" x2="20.32" y2="50.8" width="0.1524" layer="91"/>
-<junction x="22.86" y="50.8"/>
-<pinref part="SW1" gate="G$1" pin="1"/>
+<wire x1="22.86" y1="53.34" x2="22.86" y2="60.96" width="0.1524" layer="91"/>
+<wire x1="22.86" y1="53.34" x2="22.86" y2="50.8" width="0.1524" layer="91"/>
+<junction x="22.86" y="53.34"/>
+<pinref part="J3" gate="-2" pin="S"/>
+<wire x1="22.86" y1="53.34" x2="17.78" y2="53.34" width="0.1524" layer="91"/>
+<wire x1="17.78" y1="53.34" x2="17.78" y2="55.88" width="0.1524" layer="91"/>
 </segment>
 </net>
@@
 <segment>
 <pinref part="J1" gate="-1" pin="S"/>
-<wire x1="7.62" y1="50.8" x2="5.08" y2="50.8" width="0.1524" layer="91"/>
-<pinref part="SW1" gate="G$1" pin="2"/>
+<pinref part="J3" gate="-1" pin="S"/>
+<wire x1="10.16" y1="53.34" x2="12.7" y2="53.34" width="0.1524" layer="91"/>
+<wire x1="12.7" y1="53.34" x2="12.7" y2="55.88" width="0.1524" layer="91"/>
 </segment>
 </net>

Commit message: New PCB Layout
Parts:
- removed IC1: AT-TINY85V, atmel:TINY13V-10PU
- removed J1: POWER, con-garry:332-02
- removed J2: Free, con-garry:332-02
- removed J3: SWITCH, con-garry:332-02
- removed LDR1: LDR, rcl:R-EU_V526-0
- added C1, C2: 100nF, rcl:C-EUC0603
- added G1: S8401-46, battery_holder:CR2032V
- added JP1: (no value), jumper:JP1E
- added Q1: PT15-21C/TR8, SparkFun-DiscreteSemi:PHOTOTRANSISTORPT17-21C-L41-TR8
- added R4, R5: 1k, rcl:R-EU_R0603
- added R6: 100k, rcl:R-EU_R0603
- added U$1: TINY85-20SU, avr-6:TINY25/45/85-20SU
- R1, R2, R3: value 68 -> 120; device resistor:R-EU_M2012 -> rcl:R-EU_R0603
Connections:
- removed net N$11: IC1.PB4/PCINT4/ADC2, R3.2
- removed net N$12: IC1.PB3/PCINT3/CLKI/ADC3, R2.2
- removed net N$13: IC1.PB0/PCINT0/AIN0/OC0A/MOSI, R1.2
- removed net N$14: IC1.PB2/PCINT2/SCK/ADC1/T0, LDR1.2
- removed net N$7: IC1.PB1/PCINT1/AIN1/OC0B/INT0/MISO, J2-2.S
- new net FREE: JP1.1, U$1.(ADC3)PB3
- new net LED0: R1.2, U$1.(OCP)PB1
- new net LED1: R2.2, U$1.(ADC2)PB4
- new net LED2: R3.2, U$1.(AREF)PB0
- new net LIGHT: R5.1, U$1.(ADC1)PB2
- new net RESET: R6.1, U$1.(ADC0)PB5
- net GND: now also C1.1, C2.2, G1.-, JP1.2, Q1.E, U$1.GND; no longer IC1.GND, J1-2.S, J2-1.S, LDR1.1
- net N$1: now also C1.2, Q1.C, R4.1, R5.2; no longer J1-1.S, J3-1.S
- net VCC: now also C2.1, G1.+, R4.2, R6.2, U$1.VCC; no longer IC1.VCC, J3-2.S
Other:
- note added: "LED: APDA3020SECK/J3-PF"
- moved on the sheet: D1, D2, D3, R1, R2, R3
